Commit message: RViz 中 Plan 和 Execute 失败的问题ai尝试修复

File: urdf/arm/openarm_macro.xacro (robot description, xacro)
@@ -27,5 +27,5 @@
         <xacro:openarm-kinematics-link config="${kinematics_link}" name="${name}" />
         <geometry>
-          <mesh filename="package://${description_pkg}/meshes/arm/${arm_type}/visual/${name}.dae" scale="0.001 ${0.001*reflect} 0.001" />
+          <mesh filename="package://${description_pkg}/meshes/arm/${arm_type}/visual/${name}.stl" scale="0.001 ${0.001*reflect} 0.001" />
         </geometry>
       </visual>

Commit message: Revert "RViz 中 Plan 和 Execute 失败的问题ai尝试修复"
This reverts commit 29c19c3cc2be62d5ad375539774d4e2e1d610b33.

File: urdf/arm/openarm_macro.xacro (robot description, xacro)
@@ -27,5 +27,5 @@
         <xacro:openarm-kinematics-link config="${kinematics_link}" name="${name}" />
         <geometry>
-          <mesh filename="package://${description_pkg}/meshes/arm/${arm_type}/visual/${name}.stl" scale="0.001 ${0.001*reflect} 0.001" />
+          <mesh filename="package://${description_pkg}/meshes/arm/${arm_type}/visual/${name}.dae" scale="0.001 ${0.001*reflect} 0.001" />
         </geometry>
       </visual>
