Commit message: 修复upper_body、left_side和right_side都不能正常planning的问题

File: urdf/ee/openarm_hand.xacro (robot description, xacro)
@@ -60,5 +60,5 @@
       <origin xyz="0 -0.006 0.015" rpy="0 0 0" />
       <axis xyz="0 -1 0" />
-      <limit effort="333" lower="0.0" upper="0.044" velocity="10.0" />
+      <limit effort="333" lower="-0.001" upper="0.044" velocity="10.0" />
     </joint>
     <joint name="${ee_prefix}finger_joint2" type="prismatic">
@@ -67,5 +67,5 @@
       <origin xyz="0 0.006 0.015" rpy="0 0 0" />
       <axis xyz="0 1 0" />
-      <limit effort="333" lower="0.0" upper="0.044" velocity="10.0" />
+      <limit effort="333" lower="-0.001" upper="0.044" velocity="10.0" />
       <mimic joint="${ee_prefix}finger_joint1" />
     </joint>
