Commit message: 爪子力度和速度调试成功

File: urdf/ros2_control/openarm.bimanual.ros2_control.xacro (robot description, xacro)
@@ -44,4 +44,22 @@
         </joint>
       </xacro:macro>
+      <xacro:macro name="configure_gripper_joint" params="joint_name initial_position">
+        <joint name="${joint_name}">
+          <command_interface name="position"/>
+          <command_interface name="velocity"/>
+          <command_interface name="effort"/>
+          <command_interface name="gripper_speed"/>
+          <command_interface name="gripper_force"/>
+          <state_interface name="position">
+            <param name="initial_value">${initial_position}</param>
+          </state_interface>
+          <state_interface name="velocity">
+            <param name="initial_value">0.0</param>
+          </state_interface>
+          <state_interface name="effort">
+            <param name="initial_value">0.0</param>
+          </state_interface>
+        </joint>
+      </xacro:macro>
       <xacro:configure_joint joint_name="openarm_${left_arm_prefix}joint1" initial_position="0.0"/>
       <xacro:configure_joint joint_name="openarm_${left_arm_prefix}joint2" initial_position="0.0"/>
@@ -52,5 +70,5 @@
       <xacro:configure_joint joint_name="openarm_${left_arm_prefix}joint7" initial_position="0.0"/>
       <xacro:if value="${hand}">
-        <xacro:configure_joint joint_name="openarm_${left_arm_prefix}finger_joint1" initial_position="0.0" />
+        <xacro:configure_gripper_joint joint_name="openarm_${left_arm_prefix}finger_joint1" initial_position="0.0" />
       </xacro:if>
     </ros2_control>
@@ -80,5 +98,5 @@
       <xacro:configure_joint joint_name="openarm_${right_arm_prefix}joint7" initial_position="0.0"/>
       <xacro:if value="${hand}">
-        <xacro:configure_joint joint_name="openarm_${right_arm_prefix}finger_joint1" initial_position="0.0" />
+        <xacro:configure_gripper_joint joint_name="openarm_${right_arm_prefix}finger_joint1" initial_position="0.0" />
       </xacro:if>
     </ros2_control>

File: urdf/ros2_control/openarm.ros2_control.xacro (robot description, xacro)
@@ -49,4 +49,22 @@
         </joint>
       </xacro:macro>
+      <xacro:macro name="configure_gripper_joint" params="joint_name initial_position">
+        <joint name="${joint_name}">
+            <command_interface name="position"/>
+            <command_interface name="velocity"/>
+            <command_interface name="effort"/>
+            <command_interface name="gripper_speed"/>
+            <command_interface name="gripper_force"/>
+          <state_interface name="position">
+            <param name="initial_value">${initial_position}</param>
+          </state_interface>
+          <state_interface name="velocity">
+            <param name="initial_value">0.0</param>
+          </state_interface>
+          <state_interface name="effort">
+            <param name="initial_value">0.0</param>
+          </state_interface>
+        </joint>
+      </xacro:macro>
       <xacro:configure_joint joint_name="openarm_${arm_prefix}joint1" initial_position="0.0"/>
       <xacro:configure_joint joint_name="openarm_${arm_prefix}joint2" initial_position="0.0"/>
@@ -57,5 +75,5 @@
       <xacro:configure_joint joint_name="openarm_${arm_prefix}joint7" initial_position="0.0"/>
       <xacro:if value="${hand}">
-        <xacro:configure_joint joint_name="openarm_${arm_prefix}finger_joint1" initial_position="0.0" />
+        <xacro:configure_gripper_joint joint_name="openarm_${arm_prefix}finger_joint1" initial_position="0.0" />
       </xacro:if>
     </ros2_control>
